File: PDB2019/PDB2019.sch (EAGLE design)
At the start: 43 parts, among them IC1 7805T, Q1 FQP30N06L, SW1 SPSTSWITCH, U1 LTC3807EFEPBFTSSOP-20_FE/CB-M, U2 RJK0651DPB-00J5LFPAK-M, U3 RJK0651DPB-00J5LFPAK-M, U4 BTN8982TA

Commit message: Add files via upload
Parts:
- added J1: 3-644892-8, 3-644892-8:3-644892-8
- added J2: 5-146259-6, 5-146259-6:5-146259-6
- added R13, R14, R16, R18, R20, R22, R24: 1k, eagle-ltspice:RR1210
- added R15: 2k, eagle-ltspice:RR1210
- added R17: 4k, eagle-ltspice:RR1210
- added R19: 5k, eagle-ltspice:RR1210
- added R21: 6k, eagle-ltspice:RR1210
- added R23: 7k, eagle-ltspice:RR1210
- added U$9: MOUNTINGHOLES, Holes:MOUNTINGHOLES
Connections:
- new net A1: R13.2, R14.1, U$8.A1
- new net A2: R15.2, R16.1, U$8.A2
- new net A3: R17.2, R18.1, U$8.A3
- new net A4: R19.2, R20.1, U$8.A4
- new net A5: R21.2, R22.1, U$8.A5
- new net A6: R23.2, R24.1, U$8.A6
- new net N$1: J1.1, U$8.A0
- new net N$15: J2.11, U$8.D4
- new net N$16: J2.10, U$8.D5
- new net N$17: J2.9, U$8.D6
- new net N$18: J2.8, U$8.D7
- new net N$19: J2.7, U$8.D8
- new net N$20: J2.6, U$8.D9
- new net N$21: J1.2, R13.1
- new net N$22: J1.3, R15.1
- new net N$23: J1.4, R17.1
- new net N$24: J1.5, R19.1
- new net N$25: J1.6, R21.1
- new net N$26: J1.7, R23.1
- new net N$28: J2.5, U$8.D10
- new net N$29: J2.4, U$8.D11
- new net N$30: J2.3, U$8.D12
- new net N$5: J2.12, U$8.D3
- new net RX: J2.1, U$8.RX1
- new net TX: J2.2, U$8.TX0
- net 0: now also J1.8, R14.2, R16.2, R18.2, R20.2, R22.2, R24.2, U$8.GND
- net ARDUINO_EN: now also U$8.D2; no longer U$8.D3

Commit message: Add files via upload
Completed most of the layout
Parts:
- renumbered U$1 to D1
Changed lines of the file:
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@@
 <part name="X_5" library="ngspice-simulation" library_urn="urn:adsk.eagle:library:527439" deviceset="GND" device=""/>
 <part name="C2" library="eagle-ltspice" library_urn="urn:adsk.eagle:library:217" deviceset="C" device="C1206" package3d_urn="urn:adsk.eagle:package:13279/1" value=".1uF"/>
-<part name="U$1" library="My_lbr" deviceset="MBRS1100T3G" device=""/>
+<part name="D1" library="My_lbr" deviceset="MBRS1100T3G" device=""/>
 <part name="X_6" library="ngspice-simulation" library_urn="urn:adsk.eagle:library:527439" deviceset="GND" device=""/>
 <part name="R3" library="eagle-ltspice" library_urn="urn:adsk.eagle:library:217" deviceset="R" device="0207/10" package3d_urn="urn:adsk.eagle:package:13275/1" value="10k"/>
@@
 <instance part="X_5" gate="G$1" x="35.56" y="33.02"/>
 <instance part="C2" gate="G$1" x="58.42" y="66.04" rot="R180"/>
-<instance part="U$1" gate="A" x="50.8" y="81.28" smashed="yes" rot="R270">
+<instance part="D1" gate="A" x="50.8" y="81.28" smashed="yes" rot="R270">
 <attribute name="VALUE" x="54.5338" y="73.2028" size="3.4798" layer="96" ratio="10" rot="SR0"/>
 <attribute name="NAME" x="55.6006" y="78.8924" size="3.4798" layer="95" ratio="10" rot="SR0"/>
@@
 <wire x1="12.7" y1="96.52" x2="17.78" y2="96.52" width="0.1524" layer="91"/>
 <label x="17.78" y="96.52" size="1.778" layer="95"/>
-<pinref part="U$1" gate="A" pin="2"/>
+<pinref part="D1" gate="A" pin="2"/>
 <wire x1="17.78" y1="96.52" x2="20.32" y2="96.52" width="0.1524" layer="91"/>
 <wire x1="50.8" y1="81.28" x2="50.8" y2="96.52" width="0.1524" layer="91"/>
@@
 <pinref part="C2" gate="G$1" pin="2"/>
 <wire x1="12.7" y1="71.12" x2="50.8" y2="71.12" width="0.1524" layer="91"/>
-<pinref part="U$1" gate="A" pin="1"/>
+<pinref part="D1" gate="A" pin="1"/>
 <wire x1="50.8" y1="71.12" x2="58.42" y2="71.12" width="0.1524" layer="91"/>
 <junction x="50.8" y="71.12"/>
-</segment>
-</net>
+<label x="33.02" y="71.12" size="1.778" layer="95"/>
+</segment>
+</net>
